File: plate/discipline-pcb.kicad_pcb (KiCad board)
At the start: 2 copper layers, 305.8 x 96.2 mm, 3 parts

Commit message: fix plate, new kicda version probably broke it
Parts:
- removed G***: LOGO, logos:coseyfannitutti_16mm
- removed G***: LOGO, logos:DISCIPLINE_SMALL_COPPER
- removed G***: LOGO, logos:DISCIPLINE_SMALL_MASK
Routing:
- removed copper zone on B.Cu, net (none)
- removed copper zone on F.Cu, net (none)
Other:
- outline, holes or cut-outs redrawn
- net class Default removed
