File: bottom/discipline-pcb.kicad_pcb (KiCad board)
At the start: 2 copper layers, 304.9 x 122.8 mm, 20 parts

Commit message: adjust plates
Parts:
- removed the G*** at (300.8, 132.5) (x2)
- removed the G*** at (291.2, 133.9) (x2)
Routing:
- net GND: vias 1 -> 0
Other:
- net class Default removed
